File: hardware/powerSupplies.sch (KiCad schematic (older format))
At the start: 3 parts, among them U501 MCP1755

Commit message: Updated pcb layout
Parts:
- U501: footprint (none) -> TO_SOT_Packages_SMD:SOT-23-5
Changed lines of the file:
@@
 F 0 "U501" H 4100 3300 60  0000 C CNN
 F 1 "MCP1755" H 3850 3900 60  0000 C CNN
-F 2 "" H 3450 3300 60  0000 C CNN
+F 2 "TO_SOT_Packages_SMD:SOT-23-5" H 3450 3300 60  0001 C CNN
 F 3 "" H 3450 3300 60  0000 C CNN
 	1    3450 3300
@@
 $EndComp
 $Comp
-L GND #PWR037
+L GND #PWR038
 U 1 1 57E6AE3A
 P 3950 3650
-F 0 "#PWR037" H 3950 3400 50  0001 C CNN
+F 0 "#PWR038" H 3950 3400 50  0001 C CNN
 F 1 "GND" H 3950 3500 50  0000 C CNN
 F 2 "" H 3950 3650 60  0000 C CNN
@@
 $EndComp
 $Comp
-L +5V #PWR038
+L +5V #PWR039
 U 1 1 57E6AE5A
 P 2050 2750
-F 0 "#PWR038" H 2050 2600 50  0001 C CNN
+F 0 "#PWR039" H 2050 2600 50  0001 C CNN
 F 1 "+5V" H 2050 2890 50  0000 C CNN
 F 2 "" H 2050 2750 60  0000 C CNN
@@
 $EndComp
 $Comp
-L GND #PWR039
+L GND #PWR040
 U 1 1 57E6AE88
 P 2900 3650
-F 0 "#PWR039" H 2900 3400 50  0001 C CNN
+F 0 "#PWR040" H 2900 3400 50  0001 C CNN
 F 1 "GND" H 2900 3500 50  0000 C CNN
 F 2 "" H 2900 3650 60  0000 C CNN
@@
 $EndComp
 $Comp
-L GND #PWR040
+L GND #PWR041
 U 1 1 57E6AE9C
 P 2450 3650
-F 0 "#PWR040" H 2450 3400 50  0001 C CNN
+F 0 "#PWR041" H 2450 3400 50  0001 C CNN
 F 1 "GND" H 2450 3500 50  0000 C CNN
 F 2 "" H 2450 3650 60  0000 C CNN
@@
 $EndComp
 $Comp
-L +3.3V #PWR041
+L +3.3V #PWR042
 U 1 1 57E6AEAF
 P 5000 2750
-F 0 "#PWR041" H 5000 2600 50  0001 C CNN
+F 0 "#PWR042" H 5000 2600 50  0001 C CNN
 F 1 "+3.3V" H 5000 2890 50  0000 C CNN
 F 2 "" H 5000 2750 60  0000 C CNN
